File: KiCad Files/FireboxRebooter.kicad_pcb (KiCad board)
At the start: 4 copper layers, 40 x 40 mm, 28 parts, among them J1 ICSP, J2 LED_SENSE, J3 MB_PWRBTN, J4 REAR_PWRBTN, Q1 Si2302, Q2 Si2302, Q3 Si2302, U1 ATtiny45-20SU

Commit message: Hardware Version 1.1
Fixed a little mistake
Parts:
- C1: value C -> 100nF
